File: kicad_project/Audio.kicad_sch (KiCad schematic)
At the start: 58 parts, among them J5 AudioJack4, J6 Conn_01x02, J7 Conn_01x02, U1 MAX98357A, U10 FSA2269, U11 TC7WH08FK,LJ(CT, U13 WM8524, U14 MAX4467, U15 WM8782, U16 TPA6132A2RTE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

Commit message: Initial commit
Parts:
- removed C18, C19: 220pF, Capacitor_SMD:C_0402_1005Metric, symbol Device:C
- removed R19: 680K, Resistor_SMD:R_0603_1608Metric, symbol Device:R
- removed U1: MAX98357A, Package_DFN_QFN:TQFN-16-1EP_3x3mm_P0.5mm_EP1.23x1.23mm, symbol Custom:MAX98357A
- added C15: 0.1uF, Capacitor_SMD:C_0805_2012Metric, symbol Device:C
- added C4: 220pF, Capacitor_SMD:C_0402_1005Metric, symbol Device:C
- added R3: 680K, Resistor_SMD:R_0603_1608Metric, symbol Device:R
- added U12: MAX98357A, Package_DFN_QFN:TQFN-16-1EP_3x3mm_P0.5mm_EP1.23x1.23mm, symbol Custom:MAX98357A
- C14: value 10uF -> 220pF; footprint Capacitor_SMD:C_0805_2012Metric -> Capacitor_SMD:C_0402_1005Metric; LCSC C15850 -> C1530
- C16: value 0.1uF -> 10uF; LCSC C49678 -> C15850
- J6: LCSC 0 -> (none)
- J7: LCSC (none) -> 0
Connections:
- net BCLK_DAC is gone; now on net BCLK_I2S: U13.9 (BCLK)
- net LRCLK_DAC is gone; now on net LRCLK_I2S: U13.8 (LRCLK)
- net 5V: now also C16.2, C15.1, U12.7 (VDD), U12.8 (VDD); no longer C14.2, C16.1
- net DAT_DAC: now also U12.1 (DIN)
- net GND: now also C16.1, C15.2, C4.2, U12.11 (GND), U12.15 (GND), U12.17 (EP), U12.3 (GND); no longer C16.2
- net ~{AMP_SD}: now also R3.2
- net at J7.1 (Pin_1): now also C14.2, FB1.2
- net at J7.2 (Pin_2): now also FB2.1, C4.1
- net at FB1.1: now also U12.10 (OUT-)
- net at J6.1 (Pin_1): now also U12.2 (GAIN_SLOT); no longer FB1.2
- net at J6.2 (Pin_2): now also R3.1, U12.4 (~{SD_MODE}); no longer FB2.1
- net at FB2.2: now also U12.9 (OUT+)
- net BCLK_ADC renamed BCLK_I2S
- net BCLK_I2S: now also U12.16 (BCLK)
- net LRCLK_ADC renamed LRCLK_I2S
- net LRCLK_I2S: now also U12.14 (LRCLK)
Other:
- title: Sonatino -> Sonatino - Bluetooth Audio Edition
- moved on the sheet: C20, C21, C22, C23, C24, C25, C26, C27, C28, C29, C30, C31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
